File: kicad/blavinge.kicad_pcb (KiCad board)
At the start: 2 copper layers, 260.2 x 135.7 mm, 83 parts

Commit message: Replaced PCB with one with more mounting holes, no routing
Parts:
- added _10: , MountingHole_2.2mm_M2_Pad_Via, F.Cu at (200.5, 146.4)
- added _11: , MountingHole_2.2mm_M2_Pad_Via, F.Cu at (176.6, 192.2)
- B1: moved to F.Cu
- moved _6 70.3 mm to (242.6, 147.2)
- moved _9 53.3 mm to (152.6, 146.4), turned to -20 degrees
- moved _5 51.6 mm to (110.5, 147.2)
- moved _7 48.4 mm to (163.9, 110.0)
- moved _8 41.2 mm to (189.3, 110.0)
- moved _2 17.3 mm to (272.2, 78.8)
- moved _1 13.5 mm to (80.9, 78.8)
- moved S21 12.5 mm to (283.5, 91.5)
- moved S3 12.5 mm to (69.6, 91.5)
- moved D13 12.5 mm to (134.9, 145.3)
- moved D21 12.5 mm to (284.8, 96.3)
- moved D15 12.5 mm to (147.9, 109.5)
- moved D25 12.5 mm to (251.2, 124.7)
- moved S20 12.5 mm to (288.4, 109.8)
- moved D16 12.5 mm to (121.8, 160.7)
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Routing:
- net P16: track 355.8 -> 0.00 mm, vias 1 -> 0
- net P14: track 289.4 -> 0.00 mm, vias 1 -> 0
- net P10: track 243.5 -> 0.00 mm, vias 1 -> 0
- net P21: track 226.5 -> 0.00 mm, vias 1 -> 0
- net P20: track 222.1 -> 0.00 mm, vias 1 -> 0
- net P4: track 213.4 -> 0.00 mm, vias 1 -> 0
- net P9: track 204.1 -> 0.00 mm
- net P5: track 203.0 -> 0.00 mm, vias 1 -> 0
- net P7: track 196.7 -> 0.00 mm, vias 1 -> 0
- net P19: track 177.9 -> 0.00 mm
- net P6: track 177.7 -> 0.00 mm
- net P8: track 160.1 -> 0.00 mm, vias 1 -> 0
- net GND: track 55.4 -> 0.00 mm
- net RST: track 39.1 -> 0.00 mm
- net home_thumb: track 15.4 -> 0.00 mm
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Other:
- net class Default added: clearance 0.2, trace_width 0.25, via_dia 0.8, via_drill 0.4

Commit message: Updated .gitignore, final logo
Other:
- net class Default removed
