File: kicad/blavinge.kicad_pcb (KiCad board)
At the start: 2 copper layers, 260.2 x 135.7 mm, 85 parts

Commit message: Final routing
Parts:
- B1: moved to B.Cu
- moved S29 0.27 mm to (227.1, 114.1)
- moved B1 0.27 mm to (176.4, 141.3), turned to 90 degrees
- moved S33 0.27 mm to (203.4, 104.6)
- moved S35 0.27 mm to (209.1, 170.2)
- moved S6 0.27 mm to (95.9, 85.1)
- moved S24 0.27 mm to (257.0, 85.1)
- moved _7 0.27 mm to (163.7, 109.8)
- moved D36 0.27 mm to (201.7, 193.2)
- moved D13 0.27 mm to (134.7, 145.0)
- moved S25 0.27 mm to (249.4, 119.8)
- moved D26 0.27 mm to (244.6, 106.6)
- moved D35 0.27 mm to (212.8, 173.5)
- moved S18 0.27 mm to (156.0, 192.0)
- moved D22 0.27 mm to (271.7, 125.5)
- moved D10 0.27 mm to (117.6, 136.6)
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Routing:
- net P16: track 0.00 -> 358.5 mm, vias 0 -> 1
- net P14: track 0.00 -> 289.2 mm, vias 0 -> 1
- net P10: track 0.00 -> 243.7 mm, vias 0 -> 1
- net P21: track 0.00 -> 236.9 mm
- net P4: track 0.00 -> 232.6 mm
- net P5: track 0.00 -> 226.6 mm
- net P9: track 0.00 -> 217.9 mm
- net P20: track 0.00 -> 208.6 mm
- net P7: track 0.00 -> 196.8 mm, vias 0 -> 1
- net P19: track 0.00 -> 193.7 mm
- net P6: track 0.00 -> 180.9 mm
- net P8: track 0.00 -> 159.9 mm, vias 0 -> 1
- net GND: track 0.00 -> 55.5 mm
- net RST: track 0.00 -> 39.1 mm
- net pinky_bottom: track 0.00 -> 15.4 mm
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